Commit message: Add display launch file for RViz

File: warehouse_robot_description/urdf/arm.xacro (robot description, xacro)
@@ -13,6 +13,4 @@
   <xacro:property name="gripper_width" value="0.05"/>
   <xacro:property name="gripper_height" value="0.05"/>
-    <!-- BASE FOOTPRINT (standalone test için) -->
-  <link name="base_footprint"/>
   <!-- ARM BASE LINK -->
   <link name="arm_base_link">
@@ -32,5 +30,5 @@
       <origin xyz="0 0 ${arm_base_height/2}" rpy="0 0 0"/>
     </collision>
-    <xacro:inertial_box mass="5.0" x="${arm_base_length}" y="${arm_base_width}" z="${arm_base_height}"/>
+    <xacro:inertial_box mass="0.5" x="${arm_base_length}" y="${arm_base_width}" z="${arm_base_height}"/>
   </link>
   <gazebo reference="arm_base_link">
@@ -103,10 +101,4 @@
     <material>Gazebo/Yellow</material>
   </gazebo>
-  <!-- ARM BASE JOINT (fixed, standalone test için) -->
-  <joint name="arm_base_joint" type="fixed">
-    <parent link="base_footprint"/>
-    <child link="arm_base_link"/>
-    <origin xyz="0 0 ${arm_base_height/2}" rpy="0 0 0"/>
-  </joint>
   <!-- ARM BASE → LOWERARM -->
   <joint name="arm_base_to_lower_arm" type="revolute">

File: warehouse_robot_description/urdf/common_properties.xacro (robot description, xacro)
@@ -1,3 +1,3 @@
-xml<?xml version="1.0"?>
+<?xml version="1.0"?>
 <robot xmlns:xacro="http://www.ros.org/wiki/xacro">
   <xacro:macro name="inertial_box" params="mass x y z">

Commit message: Add gazebo plugins and bridge, enable base and joint control

File: warehouse_robot_description/urdf/arm.xacro (robot description, xacro)
@@ -1,5 +1,4 @@
 <?xml version="1.0"?>
 <robot xmlns:xacro="http://www.ros.org/wiki/xacro">
-<xacro:include filename="common_properties.xacro"/>
   <!-- PROPERTIES -->
   <xacro:property name="arm_base_length" value="0.08"/>
@@ -106,5 +105,5 @@
     <child link="lower_arm_link"/>
     <origin xyz="0 0 ${arm_base_height}" rpy="0 0 0"/>
-    <axis xyz="0 1 0"/>
+    <axis xyz="0 -1 0"/>
     <limit lower="0" upper="${pi/2}" effort="100" velocity="100"/>
     <dynamics friction="0.05" damping="0.1"/>
@@ -115,5 +114,5 @@
     <child link="upper_arm_link"/>
     <origin xyz="0 0 ${lower_arm_length}" rpy="0 0 0"/>
-    <axis xyz="0 1 0"/>
+    <axis xyz="0 -1 0"/>
     <limit lower="0" upper="${pi/2}" effort="100" velocity="100"/>
     <dynamics friction="0.05" damping="0.1"/>
@@ -124,7 +123,40 @@
     <child link="gripper_link"/>
     <origin xyz="0 0 ${upper_arm_length}" rpy="0 0 0"/>
-    <axis xyz="0 1 0"/>
+    <axis xyz="0 -1 0"/>
     <limit lower="0" upper="${pi/2}" effort="100" velocity="100"/>
     <dynamics friction="0.05" damping="0.1"/>
   </joint>
+  <!-- JOINT STATE PUBLISHER (kol) -->
+  <gazebo>
+    <plugin filename="gz-sim-joint-state-publisher-system"
+            name="gz::sim::systems::JointStatePublisher">
+      <joint_name>arm_base_to_lower_arm</joint_name>
+      <joint_name>lower_arm_to_upper_arm</joint_name>
+      <joint_name>upper_arm_to_gripper</joint_name>
+    </plugin>
+  </gazebo>
+  <!-- JOINT POSITION CONTROLLER 1: lower, p_gain 4.0 -->
+  <gazebo>
+    <plugin filename="gz-sim-joint-position-controller-system"
+            name="gz::sim::systems::JointPositionController">
+      <joint_name>arm_base_to_lower_arm</joint_name>
+      <p_gain>4.0</p_gain>
+    </plugin>
+  </gazebo>
+  <!-- JOINT POSITION CONTROLLER 2: upper, p_gain 3.0 -->
+  <gazebo>
+    <plugin filename="gz-sim-joint-position-controller-system"
+            name="gz::sim::systems::JointPositionController">
+      <joint_name>lower_arm_to_upper_arm</joint_name>
+      <p_gain>3.0</p_gain>
+    </plugin>
+  </gazebo>
+  <!-- JOINT POSITION CONTROLLER 3: gripper, p_gain 2.0 -->
+  <gazebo>
+    <plugin filename="gz-sim-joint-position-controller-system"
+            name="gz::sim::systems::JointPositionController">
+      <joint_name>upper_arm_to_gripper</joint_name>
+      <p_gain>2.0</p_gain>
+    </plugin>
+  </gazebo>
 </robot>

File: warehouse_robot_description/urdf/mobile_base.xacro (robot description, xacro)
@@ -114,5 +114,25 @@
     <parent link="base_link"/>
     <child link="caster_wheel_link"/>
-    <origin xyz="${base_length/2-caster_wheel_radius} 0 ${-(base_height/2-caster_wheel_radius)}" rpy="0 0 0"/>
+    <origin xyz="${-base_length/2+caster_wheel_radius} 0 ${-(base_height/2-caster_wheel_radius)}" rpy="0 0 0"/>
   </joint>
+  <gazebo>
+    <plugin filename="gz-sim-diff-drive-system"
+            name="gz::sim::systems::DiffDrive">
+      <left_joint>left_wheel_joint</left_joint>
+      <right_joint>right_wheel_joint</right_joint>
+      <wheel_separation>${base_width+wheel_length}</wheel_separation>
+      <wheel_radius>${wheel_radius}</wheel_radius>
+      <odom_publish_frequency>10</odom_publish_frequency>
+      <frame_id>odom</frame_id>
+      <child_frame_id>base_footprint</child_frame_id>
+    </plugin>
+  </gazebo>
+  <!-- JOINT STATE PUBLISHER (tekerlekler) -->
+  <gazebo>
+    <plugin filename="gz-sim-joint-state-publisher-system"
+            name="gz::sim::systems::JointStatePublisher">
+      <joint_name>left_wheel_joint</joint_name>
+      <joint_name>right_wheel_joint</joint_name>
+    </plugin>
+  </gazebo>
   </robot>
